Commit message: simplified urdf

File: strands_morse_2dnav/scitosa5.urdf (robot description, URDF)
Before this commit: robot pr2, 4 links, 3 joints
Links:
- removed link base_bellow_link
- link base_link: geometry collision cylinder length=0.6 radius=0.2; visual cylinder length=0.6 radius=0.2
Joints:
- removed joint base_bellow_joint

Commit message: adjusted navigation parameters

File: strands_morse_2dnav/scitosa5.urdf (robot description, URDF)
Before this commit: robot scitosA5, 3 links, 2 joints
Links:
- added link kinect_link, mass 0.001
- link base_link: mass 116.0 -> 74.5
Joints:
- added joint kinect_joint: type fixed, parent base_link, child kinect_link, origin xyz=0.0 0.0 1.698 rpy=0 0 0, axis 0 0 1
- joint base_laser_joint: origin xyz=0.275 0.0 0.252 rpy=0 0 0 -> xyz=0.3 0.0 0.386 rpy=0 0 0
